File: mcu board/mcu board.kicad_sch (KiCad schematic)
At the start: 0 parts

Commit message: added libs
Parts:
- added U1: ESP32-S3-1, RMSmouse:450301014042, symbol mouseLib:ESP32-S3-1-WROOM
Connections:
- new net: U1.40 (GND), U1.41 (GND__1)
Changed lines of the file:
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@@
 	(generator_version "9.0")
 	(paper "A4")
+	(symbol
+		(lib_id "mouseLib:ESP32-S3-1-WROOM")
+		(at 124.46 69.85 0)
+		(unit 1)
+		(exclude_from_sim no)
+		(in_bom yes)
+		(on_board yes)
+		(dnp no)
+		(fields_autoplaced yes)
+		(property "Reference" "U1"
+			(at 124.46 44.45 0)
+			(effects
+				(font
+					(size 1.27 1.27)
+				)
+			)
+		)
+		(property "Value" "ESP32-S3-1"
+			(at 124.46 46.99 0)
+			(effects
+				(font
+					(size 1.27 1.27)
+				)
+			)
+		)
+		(property "Footprint" "RMSmouse:450301014042"
+			(at 124.46 69.85 0)
+			(effects
+				(font
+					(size 1.27 1.27)
+				)
+				(hide yes)
+			)
+		)
+		(property "Datasheet" ""
+			(at 124.46 69.85 0)
+			(effects
+				(font
+					(size 1.27 1.27)
+				)
+				(hide yes)
+			)
+		)
+		(property "Description" ""
+			(at 124.46 69.85 0)
+			(effects
+				(font
+					(size 1.27 1.27)
+				)
+				(hide yes)
+			)
+		)
+		(pin "18"
+		)
+		(pin "4"
+		)
+		(pin "5"
+		)
+		(pin "16"
+		)
+		(pin "21"
+		)
+		(pin "34"
+		)
+		(pin "33"
+		)
+		(pin "35"
+		)
+		(pin "36"
+		)
+		(pin "20"
+		)
+		(pin "37"
+		)
+		(pin "38"
+		)
+		(pin "31"
+		)
+		(pin "6"
+		)
+		(pin "24"
+		)
+		(pin "22"
+		)
+		(pin "28"
+		)
+		(pin "15"
+		)
+		(pin "27"
+		)
+		(pin "14"
+		)
+		(pin "32"
+		)
+		(pin "7"
+		)
+		(pin "11"
+		)
+		(pin "25"
+		)
+		(pin "1"
+		)
+		(pin "13"
+		)
+		(pin "9"
+		)
+		(pin "26"
+		)
+		(pin "8"
+		)
+		(pin "29"
+		)
+		(pin "2"
+		)
+		(pin "30"
+		)
+		(pin "41"
+		)
+		(pin "17"
+		)
+		(pin "23"
+		)
+		(pin "10"
+		)
+		(pin "19"
+		)
+		(pin "39"
+		)
+		(pin "12"
+		)
+		(pin "40"
+		)
+		(pin "3"
+		)
+		(instances
+			(project ""
+				(path "/e926887c-cd26-4f47-be51-3352b14f6743"
+					(reference "U1")
+					(unit 1)
+				)
+			)
+		)
+	)
 	(sheet_instances
 		(path "/"
