File: primary-board/primary board.kicad_pcb (KiCad board)
At the start: 4 copper layers, 92 x 82 mm, 70 parts, among them J1 USB_C, J10 Motor Connector Right, J5 I2C Breakout, J6 Conn_01x02, J7 Conn_01x02, J8 Conn_01x02, J9 Motor Connector Left, Q1 SFH 313 FA-3/4, Q2 SFH 313 FA-3/4, Q3 SFH 313 FA-3/4, Q4 SFH 313 FA-3/4, Q5 NMOS, Q6 NMOS, Q7 NMOS, Q8 NMOS, SW1 SW_SPST, SW2 SW_SPST, SW3 SW_SPDT, U1 ESP32-S3-1, U2 L7806, U3 L7806, U4 AZ1117-3.3, U5 DRV8411ARTER, U6 TLV9004xRUCR

Commit message: dante review
Connections:
- C11 pad 1: Vdrive -> +6V
- U5 pad 10: Vdrive -> +6V
Routing:
- net +6V: track 36.2 -> 41.6 mm
- net Vdrive: track 3.30 -> 0.00 mm
